Commit message: Update hsrb4s.urdf

File: robot/hsrb4s.urdf (robot description, URDF)
Before this commit: robot hsrb, 51 links, 50 joints
Joints:
- joint base_l_passive_wheel_x_frame_joint: origin xyz=0.1495                 0.055                 0.03 rpy=0.0 0.0 0.0 -> xyz=0.1495 0.055 0.03 rpy=0.0 0.0 0.0
- joint base_r_passive_wheel_x_frame_joint: origin xyz=0.1495                 -0.055                 0.03 rpy=0.0 0.0 0.0 -> xyz=0.1495 -0.055 0.03 rpy=0.0 0.0 0.0

Commit message: modify: hsr ikfast

File: robot/hsrb4s.urdf (robot description, URDF)
Before this commit: robot hsrb, 51 links, 50 joints
Links:
- link base_footprint: mass None -> 0
Joints:
- joint base_l_passive_wheel_x_frame_joint: origin xyz=0.1495                 0.055                 0.03 rpy=0.0 0.0 0.0 -> xyz=0.1495 0.055 0.03 rpy=0.0 0.0 0.0
- joint base_r_passive_wheel_x_frame_joint: origin xyz=0.1495                 -0.055                 0.03 rpy=0.0 0.0 0.0 -> xyz=0.1495 -0.055 0.03 rpy=0.0 0.0 0.0
